Commit message: nav-fixed-1

File: dynominion_rmf_description/urdf/dynominion_rmf_description.urdf.xacro (robot description, xacro)
@@ -2,5 +2,5 @@
 <robot xmlns:xacro="http://www.ros.org/wiki/xacro">
   <xacro:arg name="robot_name" default="dynominion1" />
-  <xacro:property name="robot_name" value="$(arg robot_name)/" />
+  <xacro:property name="robot_name" value="$(arg robot_name)" />
   <xacro:macro name="dynominion_rmf_base">
   <xacro:macro name="visual_collision" params="stl material">
@@ -26,11 +26,11 @@
       </collision>
   </xacro:macro>
-  <link name="${robot_name}base_footprint" />
+  <link name="base_footprint" />
   <joint name="base_joint" type="fixed">
-    <parent link="${robot_name}base_footprint"/>
-    <child link="${robot_name}base_link"/>
+    <parent link="base_footprint"/>
+    <child link="base_link"/>
     <origin xyz="0 0 0.0925" rpy="0 0 0"/>
   </joint>
-  <link name="${robot_name}base_link">
+  <link name="base_link">
     <inertial>
       <origin
@@ -54,12 +54,12 @@
       rpy="0 0 0" />
     <parent
-      link="${robot_name}base_link" />
-    <child
-      link="${robot_name}left_wheel" />
+      link="base_link" />
+    <child
+      link="left_wheel" />
     <axis
       xyz="0 1 0" />
     <dynamics damping="0.3"/>
   </joint>
-  <link name="${robot_name}left_wheel">
+  <link name="left_wheel">
     <inertial>
       <origin
@@ -83,12 +83,12 @@
       rpy="0 0 0" />
     <parent
-      link="${robot_name}base_link" />
-    <child
-      link="${robot_name}right_wheel" />
+      link="base_link" />
+    <child
+      link="right_wheel" />
     <axis
       xyz="0 1 0" />
     <dynamics damping="0.3"/>
   </joint>
-  <link name="${robot_name}right_wheel">
+  <link name="right_wheel">
     <inertial>
       <origin
@@ -107,5 +107,5 @@
     <xacro:visual_collision stl="right_wheel_l1.STL" material="wheel"/>
   </link>
-  <link name="${robot_name}laser">
+  <link name="laser">
     <inertial>
       <origin
@@ -129,11 +129,11 @@
       rpy="0 0 3.1415926535897931" />
     <parent
-      link="${robot_name}base_link" />
-    <child
-      link="${robot_name}laser" />
-    <axis
-      xyz="0 0 0" />
-  </joint>
-  <link name="${robot_name}imu_link">
+      link="base_link" />
+    <child
+      link="laser" />
+    <axis
+      xyz="0 0 0" />
+  </joint>
+  <link name="imu_link">
     <inertial>
       <origin
@@ -157,11 +157,11 @@
       rpy="0 0 0" />
     <parent
-      link="${robot_name}base_link" />
-    <child
-      link="${robot_name}imu_link" />
-    <axis
-      xyz="0 0 0" />
-  </joint>
-  <link name="${robot_name}gps"/>
+      link="base_link" />
+    <child
+      link="imu_link" />
+    <axis
+      xyz="0 0 0" />
+  </joint>
+  <link name="gps"/>
   <joint name="gps_joint" type="fixed">
     <origin
@@ -169,12 +169,12 @@
       rpy="0 0 0" />
     <parent
-      link="${robot_name}base_link" />
-    <child
-      link="${robot_name}gps" />
+      link="base_link" />
+    <child
+      link="gps" />
     <axis
       xyz="0 0 0" />
   </joint>
   <link
-    name="${robot_name}castor_1">
+    name="castor_1">
     <inertial>
       <origin
@@ -198,12 +198,12 @@
       rpy="0 0 0" />
     <parent
-      link="${robot_name}base_link" />
-    <child
-      link="${robot_name}castor_1" />
+      link="base_link" />
+    <child
+      link="castor_1" />
     <axis
       xyz="0 0 0" />
   </joint>
   <link
-    name="${robot_name}castor_2">
+    name="castor_2">
     <inertial>
       <origin
@@ -227,11 +227,11 @@
       rpy="0 0 0" />
     <parent
-      link="${robot_name}base_link" />
-    <child
-      link="${robot_name}castor_2" />
-    <axis
-      xyz="0 0 0" />
-  </joint>
-  <link name="${robot_name}castor_3">
+      link="base_link" />
+    <child
+      link="castor_2" />
+    <axis
+      xyz="0 0 0" />
+  </joint>
+  <link name="castor_3">
     <inertial>
       <origin
@@ -255,12 +255,12 @@
       rpy="0 0 0" />
     <parent
-      link="${robot_name}base_link" />
-    <child
-      link="${robot_name}castor_3" />
+      link="base_link" />
+    <child
+      link="castor_3" />
     <axis
       xyz="0 0 0" />
   </joint>
   <link
-    name="${robot_name}castor_4">
+    name="castor_4">
     <inertial>
       <origin
@@ -286,7 +286,7 @@
       rpy="0 0 0" />
     <parent
-      link="${robot_name}base_link" />
-    <child
-      link="${robot_name}castor_4" />
+      link="base_link" />
+    <child
+      link="castor_4" />
     <axis
       xyz="0 0 0" />

File: dynominion_rmf_gazebo/urdf/dynominion_rmf.urdf.xacro (robot description, xacro)
@@ -3,5 +3,5 @@
 <robot xmlns:xacro="http://www.ros.org/wiki/xacro" name="dynominion_rmf">
   <xacro:arg name="robot_name" default="dynominion1" />
-  <xacro:property name="robot_name" value="$(arg robot_name)/" />
+  <xacro:property name="robot_name" value="$(arg robot_name)" />
   <xacro:include filename="$(find dynominion_rmf_description)/urdf/dynominion_rmf_description.urdf.xacro" />
   <!-- Import Rviz colors -->

File: dynominion_rmf_gazebo/urdf/gazebo_ros2_control.xacro (robot description, xacro)
@@ -31,4 +31,5 @@
             <remapping>diff_drive_base_controller/cmd_vel:=cmd_vel</remapping>
             <remapping>diff_drive_base_controller/odom:=odom</remapping>
+            <remapping>/tf:=/tf_discard</remapping>
           </ros>
         </plugin>

File: dynominion_rmf_gazebo/urdf/gazebo_sensor_plugin.xacro (robot description, xacro)
@@ -1,5 +1,5 @@
 <?xml version="1.0"?>
 <robot xmlns:xacro="http://www.ros.org/wiki/xacro">
-    <gazebo reference ="$(arg robot_name)/imu_link">
+    <gazebo reference ="imu_link">
         <sensor name="imu_sensor" type="imu">
             <always_on>1</always_on>
@@ -7,12 +7,12 @@
             <visualize>true</visualize>
             <topic>$(arg robot_name)/imu</topic>
-            <frame_id>$(arg robot_name)/imu_link</frame_id>
+            <frame_id>imu_link</frame_id>
         </sensor>
     </gazebo>
-    <gazebo reference ="$(arg robot_name)/laser">
+    <gazebo reference ="laser">
         <sensor name='gpu_lidar' type='gpu_lidar'>
-            <pose relative_to='$(arg robot_name)/laser'>0 0 0 0 0 0</pose>
+            <pose relative_to='laser'>0 0 0 0 0 0</pose>
             <topic>$(arg robot_name)/scan</topic>
-            <frame_id>$(arg robot_name)/laser</frame_id>
+            <frame_id>laser</frame_id>
             <update_rate>10</update_rate>
             <ray>
